Commit message: code refactoring

File: urdf/gazebo.xacro (robot description, xacro)
@@ -2,19 +2,36 @@
 <robot xmlns:xacro="http://www.ros.org/wiki/xacro">
     <gazebo>
-        <plugin name="diff_drive" filename="libgazebo_ros_diff_drive.so">
-            <!-- Wheel Information -->
-            <left_joint>left_wheel_joint</left_joint>
-            <right_joint>right_wheel_joint</right_joint>
-            <wheel_separation>0.35</wheel_separation>
+        <plugin name="gazebo_ros_ackermann_drive" filename="libgazebo_ros_ackermann_drive.so">
+            <ros>
+                <remapping>cmd_vel:=cmd_vel</remapping>
+                <remapping>odom:=odom</remapping>
+                <remapping>distance:=distance</remapping>
+            </ros>
+            <update_rate>100.0</update_rate>
+            <front_left_joint>front_left_wheel_joint</front_left_joint>
+            <front_right_joint>front_right_wheel_joint</front_right_joint>
+            <rear_left_joint>rear_left_wheel_joint</rear_left_joint>
+            <rear_right_joint>rear_right_wheel_joint</rear_right_joint>
+            <left_steering_joint>front_left_steer_joint</left_steering_joint>
+            <right_steering_joint>front_right_steer_joint</right_steering_joint>
+            <wheel_separation>0.28</wheel_separation>
             <wheel_diameter>0.1</wheel_diameter>
-            <!-- Limits -->
-            <max_wheel_torque>200</max_wheel_torque>
+            <max_steer>0.6</max_steer>
+            <max_steering_angle>7.85</max_steering_angle>
+            <max_speed>2.5</max_speed>
             <max_wheel_acceleration>10.0</max_wheel_acceleration>
-            <!-- Output -->
-            <odometry_frame>odom</odometry_frame>
-            <robot_base_frame>base_link</robot_base_frame>
+            <max_wheel_torque>200.0</max_wheel_torque>
+            <left_steering_pid_gain>500.0 0.0 1.0</left_steering_pid_gain>
+            <left_steering_i_range>0 0</left_steering_i_range>
+            <right_steering_pid_gain>500.0 0.0 1.0</right_steering_pid_gain>
+            <right_steering_i_range>0 0</right_steering_i_range>
+            <linear_velocity_pid_gain>100.0 0.0 1.0</linear_velocity_pid_gain>
+            <linear_velocity_i_range>0 0</linear_velocity_i_range>
             <publish_odom>true</publish_odom>
             <publish_odom_tf>true</publish_odom_tf>
             <publish_wheel_tf>true</publish_wheel_tf>
+            <publish_distance>true</publish_distance>
+            <odometry_frame>odom</odometry_frame>
+            <robot_base_frame>base_link</robot_base_frame>
         </plugin>
     </gazebo>

File: urdf/robot.xacro (robot description, xacro)
@@ -22,5 +22,5 @@
         </collision>
         <xacro:inertial_box mass="15.0" x="0.4" y="0.2" z="0.1">
-            <origin xyz="0.2 0 -0.1" rpy="0 0 0"/>
+            <origin xyz="0.1 0 -0.1" rpy="0 0 0"/>
         </xacro:inertial_box>
     </link>
@@ -53,6 +53,6 @@
             <kp>1000000.0</kp>
             <kd>100.0</kd>
-            <mu1>1.0</mu1>
-            <mu2>1.0</mu2>
+            <mu1>2.0</mu1>
+            <mu2>2.0</mu2>
         </gazebo>
     </xacro:macro>
@@ -107,4 +107,4 @@
     <xacro:front_steer_wheel prefix="front_left" y_offset="0.14" dir="-1"/>
     <xacro:front_steer_wheel prefix="front_right" y_offset="-0.14" dir="1"/>
-    <xacro:include filename="gazebo_ackermann.xacro"/>
+    <xacro:include filename="gazebo.xacro"/>
 </robot>

Commit message: fixed nav

File: urdf/gazebo.xacro (robot description, xacro)
@@ -19,5 +19,5 @@
             <max_steer>0.6</max_steer>
             <max_steering_angle>7.85</max_steering_angle>
-            <max_speed>2.5</max_speed>
+            <max_speed>1.5</max_speed>
             <max_wheel_acceleration>10.0</max_wheel_acceleration>
             <max_wheel_torque>200.0</max_wheel_torque>
@@ -29,5 +29,5 @@
             <linear_velocity_i_range>0 0</linear_velocity_i_range>
             <publish_odom>true</publish_odom>
-            <publish_odom_tf></publish_odom_tf>
+            <publish_odom_tf>false</publish_odom_tf>
             <publish_wheel_tf>true</publish_wheel_tf>
             <publish_distance>true</publish_distance>

File: urdf/robot.xacro (robot description, xacro)
@@ -21,6 +21,6 @@
             <geometry><box size="0.4 0.2 0.1"/></geometry>
         </collision>
-        <xacro:inertial_box mass="15.0" x="0.4" y="0.2" z="0.1">
-            <origin xyz="0.1 0 -0.1" rpy="0 0 0"/>
+        <xacro:inertial_box mass="10.0" x="0.4" y="0.2" z="0.1">
+            <origin xyz="0.1 0 -0.15" rpy="0 0 0"/>
         </xacro:inertial_box>
     </link>
@@ -52,7 +52,7 @@
             <material>Gazebo/Blue</material>
             <kp>1000000.0</kp>
-            <kd>100.0</kd>
-            <mu1>2.0</mu1>
-            <mu2>2.0</mu2>
+            <kd>1.0</kd>
+            <mu1>20.0</mu1>
+            <mu2>20.0</mu2>
         </gazebo>
     </xacro:macro>
@@ -100,7 +100,7 @@
             <material>Gazebo/Blue</material>
             <kp>1000000.0</kp>
-            <kd>100.0</kd>
-            <mu1>1.0</mu1>
-            <mu2>1.0</mu2>
+            <kd>1.0</kd>
+            <mu1>20.0</mu1>
+            <mu2>20.0</mu2>
         </gazebo>
     </xacro:macro>
@@ -111,5 +111,5 @@
         <parent link="base_link"/>
         <child link="laser_frame"/>
-        <origin xyz="0.1 0 0.2" rpy="0 0 0"/>
+        <origin xyz="-0.1 0 0.2" rpy="0 0 0"/>
     </joint>
     <link name="laser_frame">
@@ -133,9 +133,9 @@
             <pose> 0 0 0 0 0 0 </pose>
             <visualize>true</visualize>
-            <update_rate>10</update_rate>
+            <update_rate>20</update_rate>
             <ray>
                 <scan>
                     <horizontal>
-                        <samples>360</samples>
+                        <samples>540</samples>
                         <min_angle>-3.14</min_angle>
                         <max_angle>3.14</max_angle>
